File: TP_FInal_V2/DSE/Kicad/kicad_ampli.kicad_pcb (KiCad board)
At the start: 2 copper layers, 141 x 118.1 mm, 110 parts, among them J1 AudioJack2, J2 Screw_Terminal_01x02, J3 Conn_01x01_Male, J3(GND)1 Conn_01x01_Male, J4 Conn_01x01_Male, J5 Conn_01x01_Male, J6 Conn_01x01_Male, J7 Conn_01x01_Male, J8 Conn_01x01_Male, Q1 BC546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

Commit message: Completando el modelo 3D de la placa.
Parts:
- Jack4, Jack5, Jack6, Jack7: footprint Connector_BarrelJack:BarrelJack_Horizontal -> Kicad-extra:BarrelJack_Horizontal_W3DM
- Q1, Q2, Q3, Q4, Q5, Q6, Q7, Q8: footprint Package_TO_SOT_THT:TO-92_Inline -> Package_TO_SOT_THT:TO-92_Inline_Wide
- RV1, RV2: footprint Potentiometer_THT:Potentiometer_ACP_CA6-H2,5_Horizontal -> Kicad-extra:Potentiometer_ACP_CA6-H2,5_Horizontal_BELOW_W3DM
- U1: footprint Package_SO:SOIC-8_3.9x4.9mm_P1.27mm -> Kicad-extra:DIP-8_W7.62mm_W3DM

Commit message: PCB 3D completo.
Parts:
- added REF**: Heatsink_150x28x59mm, Kicad-extra:Heatsink_150x28x59mm, F.Cu at (173.7, 85.0)
Changed lines of the file:
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@@
     (tracks 455)
     (zones 0)
-    (modules 110)
+    (modules 111)
     (nets 66)
   )
@@
     (add_net "Net-(U1-Pad8)")
   )
+  (module Kicad-extra:Heatsink_150x28x59mm (layer F.Cu)
+    (at 173.7 85 270)
+    (descr "Heatsink, 125x35x50mm, 3 fixation holes 3.2mm")
+    (tags heatsink)
+    (fp_text reference REF** (at 0 -34 90) (layer F.SilkS) hide
+      (effects (font (size 1 1) (thickness 0.15)))
+    )
+    (fp_text value Heatsink_150x28x59mm (at 0 4 90) (layer F.Fab) hide
+      (effects (font (size 1 1) (thickness 0.15)))
+    )
+    (fp_line (start -75 0) (end -75 -28) (layer F.SilkS) (width 0.12))
+    (fp_line (start 75 0) (end -75 0) (layer F.CrtYd) (width 0.05))
+    (fp_line (start 75 0) (end 75 -28) (layer F.CrtYd) (width 0.05))
+    (fp_line (start -75 -28) (end -75 0) (layer F.CrtYd) (width 0.05))
+    (fp_line (start -75 -28) (end 75 -28) (layer F.CrtYd) (width 0.05))
+    (fp_line (start 75 -28) (end 75 0) (layer F.Fab) (width 0.1))
+    (fp_line (start -75 0) (end 75 0) (layer F.Fab) (width 0.1))
+    (fp_line (start -75 -28) (end -75 0) (layer F.Fab) (width 0.1))
+    (fp_line (start 75 -28) (end 75 0) (layer F.SilkS) (width 0.12))
+    (fp_line (start 75 0) (end -75 0) (layer F.SilkS) (width 0.12))
+    (model ${KIPRJMOD}/3D/Heatsink_125x35x50mm_3xFixationM3_Gold.wrl
+      (offset (xyz 0 2 0))
+      (scale (xyz 0.475 0.33 0.475))
+      (rotate (xyz 0 0 0))
+    )
+  )
   (module Kicad-extra:Potentiometer_ACP_CA6-H2,5_Horizontal_BELOW_W3DM (layer F.Cu)

Commit message: Cerrando TP final.
Parts:
- J2: footprint Kicad-extra:TerminalBlock_bornier-2_P5.08mm_W3DM -> Kicad-extra:TerminalBlock_bornier-2_P5.08mm_BELOW_W3DM
Changed lines of the file:
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@@
     (add_net "Net-(U1-Pad8)")
+  )
+  (module Kicad-extra:TerminalBlock_bornier-2_P5.08mm_BELOW_W3DM (layer B.Cu)
+    (at 151.13 87.63 90)
+    (descr "simple 2-pin terminal block, pitch 5.08mm, revamped version of bornier2")
+    (tags "terminal block bornier2")
+    (fp_text reference J2 (at 2.54 5.08 270) (layer B.SilkS)
+      (effects (font (size 1 1) (thickness 0.15)) (justify mirror))
+    )
+    (fp_text value Screw_Terminal_01x02 (at 2.54 -5.08 270) (layer B.Fab)
+      (effects (font (size 1 1) (thickness 0.15)) (justify mirror))
+    )
+    (fp_text user %R (at 2.54 0 270) (layer B.Fab)
+      (effects (font (size 1 1) (thickness 0.15)) (justify mirror))
+    )
+    (fp_line (start -2.41 -2.55) (end 7.49 -2.55) (layer B.Fab) (width 0.1))
+    (fp_line (start -2.46 3.75) (end -2.46 -3.75) (layer B.Fab) (width 0.1))
+    (fp_line (start -2.46 -3.75) (end 7.54 -3.75) (layer B.Fab) (width 0.1))
+    (fp_line (start 7.54 -3.75) (end 7.54 3.75) (layer B.Fab) (width 0.1))
+    (fp_line (start 7.54 3.75) (end -2.46 3.75) (layer B.Fab) (width 0.1))
+    (fp_line (start 7.62 -2.54) (end -2.54 -2.54) (layer B.SilkS) (width 0.12))
+    (fp_line (start 7.62 -3.81) (end 7.62 3.81) (layer B.SilkS) (width 0.12))
+    (fp_line (start 7.62 3.81) (end -2.54 3.81) (layer B.SilkS) (width 0.12))
+    (fp_line (start -2.54 3.81) (end -2.54 -3.81) (layer B.SilkS) (width 0.12))
+    (fp_line (start -2.54 -3.81) (end 7.62 -3.81) (layer B.SilkS) (width 0.12))
+    (fp_line (start -2.71 4) (end 7.79 4) (layer B.CrtYd) (width 0.05))
+    (fp_line (start -2.71 4) (end -2.71 -4) (layer B.CrtYd) (width 0.05))
+    (fp_line (start 7.79 -4) (end 7.79 4) (layer B.CrtYd) (width 0.05))
+    (fp_line (start 7.79 -4) (end -2.71 -4) (layer B.CrtYd) (width 0.05))
+    (pad 1 thru_hole rect (at 0 0 90) (size 3 3) (drill 1.52) (layers *.Cu *.Mask)
+      (net 9 GND))
+    (pad 2 thru_hole circle (at 5.08 0 90) (size 3 3) (drill 1.52) (layers *.Cu *.Mask)
+      (net 23 "Net-(J2-Pad2)"))
+    (model ${KISYS3DMOD}/TerminalBlock.3dshapes/TerminalBlock_bornier-2_P5.08mm.wrl
+      (offset (xyz 2.54 0 0))
+      (scale (xyz 1 1 1))
+      (rotate (xyz 0 0 0))
+    )
+    (model "${KIPRJMOD}/3D/Terminal block 2 POS.STEP"
+      (offset (xyz 2.5 0 -0.5))
+      (scale (xyz 1 1 1))
+      (rotate (xyz 180 0 180))
+    )
   )
   (module Kicad-extra:Heatsink_150x28x59mm (layer F.Cu)
@@
       (scale (xyz 1 1 1))
       (rotate (xyz 0 0 0))
-    )
-  )
-  (module Kicad-extra:TerminalBlock_bornier-2_P5.08mm_W3DM (layer B.Cu)
-    (at 151.13 87.63 90)
-    (descr "simple 2-pin terminal block, pitch 5.08mm, revamped version of bornier2")
-    (tags "terminal block bornier2")
-    (fp_text reference J2 (at 2.54 5.08 270) (layer B.SilkS)
-      (effects (font (size 1 1) (thickness 0.15)) (justify mirror))
-    )
-    (fp_text value Screw_Terminal_01x02 (at 2.54 -5.08 270) (layer B.Fab)
-      (effects (font (size 1 1) (thickness 0.15)) (justify mirror))
-    )
-    (fp_line (start 7.79 -4) (end -2.71 -4) (layer B.CrtYd) (width 0.05))
-    (fp_line (start 7.79 -4) (end 7.79 4) (layer B.CrtYd) (width 0.05))
-    (fp_line (start -2.71 4) (end -2.71 -4) (layer B.CrtYd) (width 0.05))
-    (fp_line (start -2.71 4) (end 7.79 4) (layer B.CrtYd) (width 0.05))
-    (fp_line (start -2.54 -3.81) (end 7.62 -3.81) (layer B.SilkS) (width 0.12))
-    (fp_line (start -2.54 3.81) (end -2.54 -3.81) (layer B.SilkS) (width 0.12))
-    (fp_line (start 7.62 3.81) (end -2.54 3.81) (layer B.SilkS) (width 0.12))
-    (fp_line (start 7.62 -3.81) (end 7.62 3.81) (layer B.SilkS) (width 0.12))
-    (fp_line (start 7.62 -2.54) (end -2.54 -2.54) (layer B.SilkS) (width 0.12))
-    (fp_line (start 7.54 3.75) (end -2.46 3.75) (layer B.Fab) (width 0.1))
-    (fp_line (start 7.54 -3.75) (end 7.54 3.75) (layer B.Fab) (width 0.1))
-    (fp_line (start -2.46 -3.75) (end 7.54 -3.75) (layer B.Fab) (width 0.1))
-    (fp_line (start -2.46 3.75) (end -2.46 -3.75) (layer B.Fab) (width 0.1))
-    (fp_line (start -2.41 -2.55) (end 7.49 -2.55) (layer B.Fab) (width 0.1))
-    (fp_text user %R (at 2.54 0 270) (layer B.Fab)
-      (effects (font (size 1 1) (thickness 0.15)) (justify mirror))
-    )
-    (pad 2 thru_hole circle (at 5.08 0 90) (size 3 3) (drill 1.52) (layers *.Cu *.Mask)
-      (net 23 "Net-(J2-Pad2)"))
-    (pad 1 thru_hole rect (at 0 0 90) (size 3 3) (drill 1.52) (layers *.Cu *.Mask)
-      (net 9 GND))
-    (model ${KISYS3DMOD}/TerminalBlock.3dshapes/TerminalBlock_bornier-2_P5.08mm.wrl
-      (offset (xyz 2.539999961853027 0 0))
-      (scale (xyz 1 1 1))
-      (rotate (xyz 0 0 0))
-    )
-    (model "${KIPRJMOD}/3D/Terminal block 2 POS.STEP"
-      (offset (xyz 2.5 0 0))
-      (scale (xyz 1 1 1))
-      (rotate (xyz 0 0 0))
