File: TP_FInal_V2/DSE/Kicad/kicad_ampli.sch (KiCad schematic (older format))
At the start: 108 parts, among them J1 AudioJack2, J2 Screw_Terminal_01x02, J3 Conn_01x01_Male, J3(GND)1 Conn_01x01_Male, J4 Conn_01x01_Male, J5 Conn_01x01_Male, J6 Conn_01x01_Male, J7 Conn_01x01_Male, J8 Conn_01x01_Male, Q1 BC546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

Commit message: Completando el modelo 3D de la placa.
Parts:
- U1: value LMH6609MA -> NE5532; footprint Package_SO:SOIC-8_3.9x4.9mm_P1.27mm -> Kicad-extra:DIP-8_W7.62mm_W3DM; symbol Amplifier_Operational:LMH6609MA -> Amplifier_Operational:NE5532
Connections:
- net at C10.1, C14.1, C24.1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: no longer U1.7 (V+)
- net at C11.1, C15.2, C25.2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: no longer U1.4 (V-)
- net at C18.1, C19.1, R27.2: now also U1.1; no longer U1.6
Changed lines of the file:
@@
 	3000 6000 3000 6500
 $Comp
-L Amplifier_Operational:LMH6609MA U1
+L Amplifier_Operational:NE5532 U1
 U 1 1 5D17A951
 P 2700 6000
 F 0 "U1" H 3044 6046 50  0000 L CNN
-F 1 "LMH6609MA" H 3044 5955 50  0000 L CNN
-F 2 "Package_SO:SOIC-8_3.9x4.9mm_P1.27mm" H 2600 5800 50  0001 L CNN
-F 3 "http://www.ti.com/lit/ds/symlink/lmh6609.pdf" H 2850 6150 50  0001 C CNN
+F 1 "NE5532" H 3044 5955 50  0000 L CNN
+F 2 "Kicad-extra:DIP-8_W7.62mm_W3DM" H 2600 5800 50  0001 L CNN
+F 3 "NE5532" H 2850 6150 50  0001 C CNN
 	1    2700 6000
 	1    0    0    -1

Commit message: PCB 3D completo.
Parts:
- Jack4, Jack5, Jack6, Jack7: footprint Kicad-extra:BarrelJack_Horizontal_W3DM -> Connector_BarrelJack:BarrelJack_Horizontal
- U1: value NE5532 -> LMH6609MA; footprint Kicad-extra:DIP-8_W7.62mm_W3DM -> Package_SO:SOIC-8_3.9x4.9mm_P1.27mm; symbol Amplifier_Operational:NE5532 -> Amplifier_Operational:LMH6609MA
Connections:
- net at C10.1, C14.1, C24.1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: now also U1.7 (V+)
- net at C11.1, C15.2, C25.2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: now also U1.4 (V-)
- net at C18.1, C19.1, R27.2: now also U1.6; no longer U1.1
Changed lines of the file:
@@
 encoding utf-8
 Sheet 1 1
-Title "Proyecto de diseño de circuitos electrónicos"
-Date "2019-07-14"
-Rev "1.1"
-Comp "FIUBA"
+Title ""
+Date ""
+Rev ""
+Comp ""
 Comment1 ""
 Comment2 ""
@@
 	3000 6000 3000 6500
 $Comp
-L Amplifier_Operational:NE5532 U1
+L Amplifier_Operational:LMH6609MA U1
 U 1 1 5D17A951
 P 2700 6000
 F 0 "U1" H 3044 6046 50  0000 L CNN
-F 1 "NE5532" H 3044 5955 50  0000 L CNN
-F 2 "Kicad-extra:DIP-8_W7.62mm_W3DM" H 2600 5800 50  0001 L CNN
-F 3 "NE5532" H 2850 6150 50  0001 C CNN
+F 1 "LMH6609MA" H 3044 5955 50  0000 L CNN
+F 2 "Package_SO:SOIC-8_3.9x4.9mm_P1.27mm" H 2600 5800 50  0001 L CNN
+F 3 "http://www.ti.com/lit/ds/symlink/lmh6609.pdf" H 2850 6150 50  0001 C CNN
 	1    2700 6000
 	1    0    0    -1
@@
 F 0 "Jack4" H 9820 3008 50  0000 R CNN
 F 1 "+15" H 9820 3099 50  0000 R CNN
-F 2 "Kicad-extra:BarrelJack_Horizontal_W3DM" H 10100 3010 50  0001 C CNN
+F 2 "Connector_BarrelJack:BarrelJack_Horizontal" H 10100 3010 50  0001 C CNN
 F 3 "~" H 10100 3010 50  0001 C CNN
 	1    10050 3050
@@
 F 0 "Jack5" H 9820 3550 50  0000 R CNN
 F 1 "-15" H 9820 3459 50  0000 R CNN
-F 2 "Kicad-extra:BarrelJack_Horizontal_W3DM" H 10100 3460 50  0001 C CNN
+F 2 "Connector_BarrelJack:BarrelJack_Horizontal" H 10100 3460 50  0001 C CNN
 F 3 "~" H 10100 3460 50  0001 C CNN
 	1    10050 3500
@@
 F 0 "Jack7" H 10570 3500 50  0000 R CNN
 F 1 "-30" H 10570 3409 50  0000 R CNN
-F 2 "Kicad-extra:BarrelJack_Horizontal_W3DM" H 10850 3410 50  0001 C CNN
+F 2 "Connector_BarrelJack:BarrelJack_Horizontal" H 10850 3410 50  0001 C CNN
 F 3 "~" H 10850 3410 50  0001 C CNN
 	1    10800 3450
@@
 F 0 "Jack6" H 10570 3008 50  0000 R CNN
 F 1 "+30" H 10570 3099 50  0000 R CNN
-F 2 "Kicad-extra:BarrelJack_Horizontal_W3DM" H 10850 3010 50  0001 C CNN
+F 2 "Connector_BarrelJack:BarrelJack_Horizontal" H 10850 3010 50  0001 C CNN
 F 3 "~" H 10850 3010 50  0001 C CNN
 	1    10800 3050

Commit message: Correcciones.
Parts:
- RV1, RV2: footprint Potentiometer_THT:Potentiometer_ACP_CA6-H2,5_Horizontal -> Kicad-extra:Potentiometer_ACP_CA6-H2,5_Horizontal_BELOW_W3DM
Changed lines of the file:
@@
 F 0 "RV2" H 5431 3496 50  0000 R CNN
 F 1 "R_POT 2k" H 5431 3405 50  0000 R CNN
-F 2 "Potentiometer_THT:Potentiometer_ACP_CA6-H2,5_Horizontal" H 5500 3450 50  0001 C CNN
+F 2 "Kicad-extra:Potentiometer_ACP_CA6-H2,5_Horizontal_BELOW_W3DM" H 5500 3450 50  0001 C CNN
 F 3 "~" H 5500 3450 50  0001 C CNN
 	1    5500 3450
@@
 F 0 "RV1" H 3881 3546 50  0000 R CNN
 F 1 "R_POT (1k)" H 3881 3455 50  0000 R CNN
-F 2 "Potentiometer_THT:Potentiometer_ACP_CA6-H2,5_Horizontal" H 3950 3500 50  0001 C CNN
+F 2 "Kicad-extra:Potentiometer_ACP_CA6-H2,5_Horizontal_BELOW_W3DM" H 3950 3500 50  0001 C CNN
 F 3 "~" H 3950 3500 50  0001 C CNN
 	1    3950 3500

Commit message: Cerrando TP final.
Parts:
- J2: footprint Kicad-extra:TerminalBlock_bornier-2_P5.08mm_W3DM -> Kicad-extra:TerminalBlock_bornier-2_P5.08mm_BELOW_W3DM
Changed lines of the file:
@@
 $EndComp
-Wire Wire Line
-	6000 4350 6000 4400
 Wire Wire Line
 	7000 3750 7150 3750
@@
 	6000 3950 6000 4050
 Wire Wire Line
-	6000 4400 5100 4400
-Wire Wire Line
 	5100 4400 5100 3850
 Wire Wire Line
 	5100 3850 4450 3850
-Connection ~ 6000 4400
-Wire Wire Line
-	6000 4400 6000 4600
 $Comp
 L Device:R R16
@@
 F 0 "J2" H 8880 3292 50  0000 L CNN
 F 1 "Screw_Terminal_01x02" H 8880 3201 50  0000 L CNN
-F 2 "Kicad-extra:TerminalBlock_bornier-2_P5.08mm_W3DM" H 8800 3300 50  0001 C CNN
+F 2 "Kicad-extra:TerminalBlock_bornier-2_P5.08mm_BELOW_W3DM" H 8800 3300 50  0001 C CNN
 F 3 "~" H 8800 3300 50  0001 C CNN
 	1    8800 3300
@@
 Wire Wire Line
 	6600 3950 6700 3950
+Connection ~ 6000 4400
+Wire Wire Line
+	6000 4400 6000 4600
+Wire Wire Line
+	6000 4350 6000 4400
+Wire Wire Line
+	6000 4400 5100 4400
 $EndSCHEMATC
